Commit message: Update iiwa14.xacro
(cherry picked from commit 719a24448c7a4ec26a6f19522d05fa74e27df4a3)

File: lbr_description/urdf/iiwa14/iiwa14.xacro (robot description, xacro)
@@ -11,4 +11,9 @@
     <!-- KDL requires a link without inertia -->
     <link name="$(arg robot_name)_floating_link" />
+    <link name="world" />
+    <joint name="$world_to_base" type="fixed">
+        <parent link="world" />
+        <child link="$(arg robot_name)_floating_link" />
+    </joint>
     <!--joint
         between <robot_name>_floating_link and robot_name_link_0-->

Commit message: removes default tfs from launch files (#263)
(cherry picked from commit c5cf92cc108636833e49ab93efdcbc04f7e72733)

File: lbr_description/urdf/iiwa14/iiwa14.xacro (robot description, xacro)
@@ -9,15 +9,11 @@
         name="system_config_path"
         default="$(find lbr_description)/ros2_control/lbr_system_config.yaml" />
-    <!-- KDL requires a link without inertia -->
-    <link name="$(arg robot_name)_floating_link" />
+    <!-- KDL requires a link without inertia / Gazebo requires a connection to world link or robot
+    will tipple: https://github.com/lbr-stack/lbr_fri_ros2_stack/issues/230 -->
     <link name="world" />
-    <joint name="$world_to_base" type="fixed">
+    <!--joint
+        between <robot_name>_world_link and robot_name_link_0-->
+    <joint name="$(arg robot_name)_world_joint" type="fixed">
         <parent link="world" />
-        <child link="$(arg robot_name)_floating_link" />
-    </joint>
-    <!--joint
-        between <robot_name>_floating_link and robot_name_link_0-->
-    <joint name="$(arg robot_name)_floating_joint" type="fixed">
-        <parent link="$(arg robot_name)_floating_link" />
         <child link="$(arg robot_name)_link_0" />
     </joint>

File: lbr_description/urdf/iiwa7/iiwa7.xacro (robot description, xacro)
@@ -9,15 +9,11 @@
         name="system_config_path"
         default="$(find lbr_description)/ros2_control/lbr_system_config.yaml" />
-    <!-- KDL requires a link without inertia -->
-    <link name="$(arg robot_name)_floating_link" />
+    <!-- KDL requires a link without inertia / Gazebo requires a connection to world link or robot
+    will tipple: https://github.com/lbr-stack/lbr_fri_ros2_stack/issues/230 -->
     <link name="world" />
-    <joint name="$world_to_base" type="fixed">
+    <!--joint
+        between <robot_name>_world_link and robot_name_link_0-->
+    <joint name="$(arg robot_name)_world_joint" type="fixed">
         <parent link="world" />
-        <child link="$(arg robot_name)_floating_link" />
-    </joint>
-    <!--joint
-        between <robot_name>_floating_link and robot_name_link_0-->
-    <joint name="$(arg robot_name)_floating_joint" type="fixed">
-        <parent link="$(arg robot_name)_floating_link" />
         <child link="$(arg robot_name)_link_0" />
     </joint>

File: lbr_description/urdf/med14/med14.xacro (robot description, xacro)
@@ -9,15 +9,11 @@
         name="system_config_path"
         default="$(find lbr_description)/ros2_control/lbr_system_config.yaml" />
-    <!-- KDL requires a link without inertia -->
-    <link name="$(arg robot_name)_floating_link" />
+    <!-- KDL requires a link without inertia / Gazebo requires a connection to world link or robot
+    will tipple: https://github.com/lbr-stack/lbr_fri_ros2_stack/issues/230 -->
     <link name="world" />
-    <joint name="$world_to_base" type="fixed">
+    <!--joint
+        between <robot_name>_world_link and robot_name_link_0-->
+    <joint name="$(arg robot_name)_world_joint" type="fixed">
         <parent link="world" />
-        <child link="$(arg robot_name)_floating_link" />
-    </joint>
-    <!--joint
-        between <robot_name>_floating_link and robot_name_link_0-->
-    <joint name="$(arg robot_name)_floating_joint" type="fixed">
-        <parent link="$(arg robot_name)_floating_link" />
         <child link="$(arg robot_name)_link_0" />
     </joint>

File: lbr_description/urdf/med7/med7.xacro (robot description, xacro)
@@ -9,15 +9,11 @@
         name="system_config_path"
         default="$(find lbr_description)/ros2_control/lbr_system_config.yaml" />
-    <!-- KDL requires a link without inertia -->
-    <link name="$(arg robot_name)_floating_link" />
+    <!-- KDL requires a link without inertia / Gazebo requires a connection to world link or robot
+    will tipple: https://github.com/lbr-stack/lbr_fri_ros2_stack/issues/230 -->
     <link name="world" />
-    <joint name="$world_to_base" type="fixed">
+    <!--joint
+        between <robot_name>_world_link and robot_name_link_0-->
+    <joint name="$(arg robot_name)_world_joint" type="fixed">
         <parent link="world" />
-        <child link="$(arg robot_name)_floating_link" />
-    </joint>
-    <!--joint
-        between <robot_name>_floating_link and robot_name_link_0-->
-    <joint name="$(arg robot_name)_floating_joint" type="fixed">
-        <parent link="$(arg robot_name)_floating_link" />
         <child link="$(arg robot_name)_link_0" />
     </joint>
