Commit message: typo / naming / formatting (#284)
(cherry picked from commit b3dd7da175cb3b2d97b28deb059747ccee0756ad)

File: lbr_description/ros2_control/lbr_system_interface.xacro (robot description, xacro)
@@ -2,11 +2,11 @@
 <robot xmlns:xacro="http://www.ros.org/wiki/xacro">
     <xacro:macro name="lbr_system_interface"
-        params="robot_name mode joint_limits system_config_path initial_positions_path">
+        params="robot_name mode joint_limits system_config_path initial_joint_positions_path">
         <!-- load system parameters via yaml -->
         <xacro:property name="system_config"
             value="${xacro.load_yaml(system_config_path)}" />
-          <!-- load initial positions via yaml for mock/gazebo simulation -->
-        <xacro:property name="initial_positions"
-            value="${xacro.load_yaml(initial_positions_path)}" />
+        <!-- load initial positions via yaml for mock/gazebo simulation -->
+        <xacro:property name="initial_joint_positions"
+            value="${xacro.load_yaml(initial_joint_positions_path)}" />
         <ros2_control name="${robot_name}_system_interface" type="system">
             <!-- load plugin depending on mode -->
@@ -131,5 +131,5 @@
                 max_torque="${joint_limits['A1']['effort']}"
                 mode="${mode}"
-                initial_position="${initial_positions['A1'] * PI / 180}" />
+                initial_position="${initial_joint_positions['A1'] * PI / 180}" />
             <xacro:joint_interface name="${robot_name}_A2"
                 min_position="${joint_limits['A2']['lower'] * PI / 180}"
@@ -138,5 +138,5 @@
                 max_torque="${joint_limits['A2']['effort']}"
                 mode="${mode}"
-                initial_position="${initial_positions['A2'] * PI / 180}" />
+                initial_position="${initial_joint_positions['A2'] * PI / 180}" />
             <xacro:joint_interface name="${robot_name}_A3"
                 min_position="${joint_limits['A3']['lower'] * PI / 180}"
@@ -145,5 +145,5 @@
                 max_torque="${joint_limits['A3']['effort']}"
                 mode="${mode}"
-                initial_position="${initial_positions['A3'] * PI / 180}" />
+                initial_position="${initial_joint_positions['A3'] * PI / 180}" />
             <xacro:joint_interface name="${robot_name}_A4"
                 min_position="${joint_limits['A4']['lower'] * PI / 180}"
@@ -152,5 +152,5 @@
                 max_torque="${joint_limits['A4']['effort']}"
                 mode="${mode}"
-                initial_position="${initial_positions['A4'] * PI / 180}"/>
+                initial_position="${initial_joint_positions['A4'] * PI / 180}"/>
             <xacro:joint_interface name="${robot_name}_A5"
                 min_position="${joint_limits['A5']['lower'] * PI / 180}"
@@ -159,5 +159,5 @@
                 max_torque="${joint_limits['A5']['effort']}"
                 mode="${mode}"
-                initial_position="${initial_positions['A5'] * PI / 180}"/>
+                initial_position="${initial_joint_positions['A5'] * PI / 180}"/>
             <xacro:joint_interface name="${robot_name}_A6"
                 min_position="${joint_limits['A6']['lower'] * PI / 180}"
@@ -166,5 +166,5 @@
                 max_torque="${joint_limits['A6']['effort']}"
                 mode="${mode}"
-                initial_position="${initial_positions['A6'] * PI / 180}" />
+                initial_position="${initial_joint_positions['A6'] * PI / 180}" />
             <xacro:joint_interface name="${robot_name}_A7"
                 min_position="${joint_limits['A7']['lower'] * PI / 180}"
@@ -173,5 +173,5 @@
                 max_torque="${joint_limits['A7']['effort']}"
                 mode="${mode}"
-                initial_position="${initial_positions['A7'] * PI / 180}" />
+                initial_position="${initial_joint_positions['A7'] * PI / 180}" />
         </ros2_control>
     </xacro:macro>

File: lbr_description/urdf/iiwa14/iiwa14.xacro (robot description, xacro)
@@ -10,6 +10,6 @@
         default="$(find lbr_description)/ros2_control/lbr_system_config.yaml" />
     <xacro:arg
-        name="initial_positions_path"
-        default="$(find lbr_description)/ros2_control/initial_positions.yaml" />
+        name="initial_joint_positions_path"
+        default="$(find lbr_description)/ros2_control/initial_joint_positions.yaml" />
     <!-- KDL requires a link without inertia / Gazebo requires a connection to world link or robot
     will tipple https://github.com/lbr-stack/lbr_fri_ros2_stack/issues/230 -->
@@ -26,4 +26,4 @@
         mode="$(arg mode)"
         system_config_path="$(arg system_config_path)"
-        initial_positions_path="$(arg initial_positions_path)" />
+        initial_joint_positions_path="$(arg initial_joint_positions_path)" />
 </robot>

File: lbr_description/urdf/iiwa14/iiwa14_description.xacro (robot description, xacro)
@@ -3,5 +3,5 @@
     <!-- robot as extracted via https://github.com/syuntoku14/fusion2urdf -->
     <xacro:macro name="iiwa14"
-        params="robot_name:=^|lbr mode:=^|mock system_config_path:=^|'$(find lbr_description)/ros2_control/lbr_system_config.yaml' initial_positions_path:=^|'$(find lbr_description)/ros2_control/initial_positions.yaml'">
+        params="robot_name:=^|lbr mode:=^|mock system_config_path:=^|'$(find lbr_description)/ros2_control/lbr_system_config.yaml' initial_joint_positions_path:=^|'$(find lbr_description)/ros2_control/initial_joint_positions.yaml'">
         <!-- includes -->
         <xacro:include filename="$(find lbr_description)/gazebo/lbr_gazebo.xacro" />
@@ -22,5 +22,5 @@
             joint_limits="${joint_limits}"
             system_config_path="${system_config_path}"
-            initial_positions_path="${initial_positions_path}" />
+            initial_joint_positions_path="${initial_joint_positions_path}" />
         <link name="${robot_name}_link_0">
             <inertial>

File: lbr_description/urdf/iiwa7/iiwa7.xacro (robot description, xacro)
@@ -10,6 +10,6 @@
         default="$(find lbr_description)/ros2_control/lbr_system_config.yaml" />
     <xacro:arg
-        name="initial_positions_path"
-        default="$(find lbr_description)/ros2_control/initial_positions.yaml" />
+        name="initial_joint_positions_path"
+        default="$(find lbr_description)/ros2_control/initial_joint_positions.yaml" />
     <!-- KDL requires a link without inertia / Gazebo requires a connection to world link or robot
     will tipple https://github.com/lbr-stack/lbr_fri_ros2_stack/issues/230 -->
@@ -26,4 +26,4 @@
         mode="$(arg mode)"
         system_config_path="$(arg system_config_path)"
-        initial_positions_path="$(arg initial_positions_path)" />
+        initial_joint_positions_path="$(arg initial_joint_positions_path)" />
 </robot>

File: lbr_description/urdf/iiwa7/iiwa7_description.xacro (robot description, xacro)
@@ -3,5 +3,5 @@
     <!-- robot as extracted via https://github.com/syuntoku14/fusion2urdf -->
     <xacro:macro name="iiwa7"
-        params="robot_name:=^|lbr mode:=^|mock system_config_path:=^|'$(find lbr_description)/ros2_control/lbr_system_config.yaml' initial_positions_path:=^|'$(find lbr_description)/ros2_control/initial_positions.yaml'">
+        params="robot_name:=^|lbr mode:=^|mock system_config_path:=^|'$(find lbr_description)/ros2_control/lbr_system_config.yaml' initial_joint_positions_path:=^|'$(find lbr_description)/ros2_control/initial_joint_positions.yaml'">
         <!-- includes -->
         <xacro:include filename="$(find lbr_description)/gazebo/lbr_gazebo.xacro" />
@@ -22,5 +22,5 @@
             joint_limits="${joint_limits}"
             system_config_path="${system_config_path}"
-            initial_positions_path="${initial_positions_path}" />
+            initial_joint_positions_path="${initial_joint_positions_path}" />
         <link name="${robot_name}_link_0">
             <inertial>

File: lbr_description/urdf/med14/med14.xacro (robot description, xacro)
@@ -10,6 +10,6 @@
         default="$(find lbr_description)/ros2_control/lbr_system_config.yaml" />
     <xacro:arg
-        name="initial_positions_path"
-        default="$(find lbr_description)/ros2_control/initial_positions.yaml" />
+        name="initial_joint_positions_path"
+        default="$(find lbr_description)/ros2_control/initial_joint_positions.yaml" />
     <!-- KDL requires a link without inertia / Gazebo requires a connection to world link or robot
     will tipple https://github.com/lbr-stack/lbr_fri_ros2_stack/issues/230 -->
@@ -26,4 +26,4 @@
         mode="$(arg mode)"
         system_config_path="$(arg system_config_path)"
-        initial_positions_path="$(arg initial_positions_path)" />
+        initial_joint_positions_path="$(arg initial_joint_positions_path)" />
 </robot>

File: lbr_description/urdf/med14/med14_description.xacro (robot description, xacro)
@@ -3,5 +3,5 @@
     <!-- robot as extracted via https://github.com/syuntoku14/fusion2urdf -->
     <xacro:macro name="med14"
-        params="robot_name:=^|lbr mode:=^|mock system_config_path:=^|'$(find lbr_description)/ros2_control/lbr_system_config.yaml' initial_positions_path:=^|'$(find lbr_description)/ros2_control/initial_positions.yaml'">
+        params="robot_name:=^|lbr mode:=^|mock system_config_path:=^|'$(find lbr_description)/ros2_control/lbr_system_config.yaml' initial_joint_positions_path:=^|'$(find lbr_description)/ros2_control/initial_joint_positions.yaml'">
         <!-- includes -->
         <xacro:include filename="$(find lbr_description)/gazebo/lbr_gazebo.xacro" />
@@ -22,5 +22,5 @@
             joint_limits="${joint_limits}"
             system_config_path="${system_config_path}"
-            initial_positions_path="${initial_positions_path}" />
+            initial_joint_positions_path="${initial_joint_positions_path}" />
         <link name="${robot_name}_link_0">
             <inertial>

File: lbr_description/urdf/med7/med7.xacro (robot description, xacro)
@@ -10,6 +10,6 @@
         default="$(find lbr_description)/ros2_control/lbr_system_config.yaml" />
     <xacro:arg
-        name="initial_positions_path"
-        default="$(find lbr_description)/ros2_control/initial_positions.yaml" />
+        name="initial_joint_positions_path"
+        default="$(find lbr_description)/ros2_control/initial_joint_positions.yaml" />
     <!-- KDL requires a link without inertia / Gazebo requires a connection to world link or robot
     will tipple https://github.com/lbr-stack/lbr_fri_ros2_stack/issues/230 -->
@@ -26,4 +26,4 @@
         mode="$(arg mode)"
         system_config_path="$(arg system_config_path)"
-        initial_positions_path="$(arg initial_positions_path)" />
+        initial_joint_positions_path="$(arg initial_joint_positions_path)" />
 </robot>

File: lbr_description/urdf/med7/med7_description.xacro (robot description, xacro)
@@ -3,5 +3,5 @@
     <!-- robot as extracted via https://github.com/syuntoku14/fusion2urdf -->
     <xacro:macro name="med7"
-        params="robot_name:=^|lbr mode:=^|mock system_config_path:=^|'$(find lbr_description)/ros2_control/lbr_system_config.yaml' initial_positions_path:=^|'$(find lbr_description)/ros2_control/initial_positions.yaml'">
+        params="robot_name:=^|lbr mode:=^|mock system_config_path:=^|'$(find lbr_description)/ros2_control/lbr_system_config.yaml' initial_joint_positions_path:=^|'$(find lbr_description)/ros2_control/initial_joint_positions.yaml'">
         <!-- includes -->
         <xacro:include filename="$(find lbr_description)/gazebo/lbr_gazebo.xacro" />
@@ -22,5 +22,5 @@
             joint_limits="${joint_limits}"
             system_config_path="${system_config_path}"
-            initial_positions_path="${initial_positions_path}" />
+            initial_joint_positions_path="${initial_joint_positions_path}" />
         <!-- properties -->
         <link name="${robot_name}_link_0">
